Commit message: change source

File: urdf/kr210l150_link.urdf (robot description, URDF)
Before this commit: robot kuka_kr210, 8 links, 7 joints
Links:
- link base_link: geometry collision mesh filename=C:/Users/whj03/Desktop/admittance/urdf/meshes/kr210l150/col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; visual mesh filename=C:/Users/whj03/Desktop/admittance/urdf/meshes/kr210l150/vis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
- link link_1: geometry collision mesh filename=C:/Users/whj03/Desktop/admittance/urdf/meshes/kr210l150/col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; visual mesh filename=C:/Users/whj03/Desktop/admittance/urdf/meshes/kr210l150/vis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
- link link_2: geometry collision mesh filename=C:/Users/whj03/Desktop/admittance/urdf/meshes/kr210l150/col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; visual mesh filename=C:/Users/whj03/Desktop/admittance/urdf/meshes/kr210l150/vis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
- link link_3: geometry collision mesh filename=C:/Users/whj03/Desktop/admittance/urdf/meshes/kr210l150/col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; visual mesh filename=C:/Users/whj03/Desktop/admittance/urdf/meshes/kr210l150/vis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
- link link_4: geometry collision mesh filename=C:/Users/whj03/Desktop/admittance/urdf/meshes/kr210l150/col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; visual mesh filename=C:/Users/whj03/Desktop/admittance/urdf/meshes/kr210l150/vis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
- link link_5: geometry collision mesh filename=C:/Users/whj03/Desktop/admittance/urdf/meshes/kr210l150/col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; visual mesh filename=C:/Users/whj03/Desktop/admittance/urdf/meshes/kr210l150/vis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
- link link_6: geometry collision mesh filename=C:/Users/whj03/Desktop/admittance/urdf/meshes/kr210l150/col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; visual mesh filename=C:/Users/whj03/Desktop/admittance/urdf/meshes/kr210l150/vis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

Commit message: change source

File: urdf/kr210l150_link.urdf (robot description, URDF)
Before this commit: robot kuka_kr210, 8 links, 7 joints
Links:
- added link eef
- added link rail_link, mass 400.0; collision mesh filename=C:/Users/whj03/Desktop/admittance/urdf/rail.stl; visual mesh filename=C:/Users/whj03/Desktop/admittance/urdf/rail.stl
- link base_link: geometry collision mesh filename=C:/Users/whj03/Desktop/admittance/urdf/meshes/kr210l150/col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; visual mesh filename=C:/Users/whj03/Desktop/admittance/urdf/meshes/kr210l150/col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
- link link_1: geometry collision mesh filename=C:/Users/whj03/Desktop/admittance/urdf/meshes/kr210l150/col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; visual mesh filename=C:/Users/whj03/Desktop/admittance/urdf/meshes/kr210l150/col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
- link link_3: geometry collision mesh filename=C:/Users/whj03/Desktop/admittance/urdf/meshes/kr210l150/col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; visual mesh filename=C:/Users/whj03/Desktop/admittance/urdf/meshes/kr210l150/col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
- link link_4: geometry collision mesh filename=C:/Users/whj03/Desktop/admittance/urdf/meshes/kr210l150/col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; visual mesh filename=C:/Users/whj03/Desktop/admittance/urdf/meshes/kr210l150/col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
- link link_5: geometry collision mesh filename=C:/Users/whj03/Desktop/admittance/urdf/meshes/kr210l150/col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; visual mesh filename=C:/Users/whj03/Desktop/admittance/urdf/meshes/kr210l150/col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
Joints:
- added joint r_fixed_eef: type fixed, parent link_6, child eef, origin xyz=0 0 0 rpy=0 0 0, axis 0 0 1
- added joint rail_joint: type prismatic, parent rail_link, child base_link, origin xyz=0.0 0.0 0.38, axis 1 0 0, limit lower=-3.5 upper=3.5 effort=1000.0 velocity=5
- joint world_fixed: child base_link -> rail_link
