Commit message: change source

File: urdf/TFtest.urdf (robot description, URDF)
Before this commit: robot box, 2 links, 1 joints
Links:
- removed link box
- added link end_link, mass 1; collision box size=0.3 0.3 0.3; visual box size=0.3 0.3 0.3
Joints:
- joint world_fixed: child box -> end_link

File: urdf/box.urdf (robot description, URDF)
Before this commit: robot box, 2 links, 1 joints
Links:
- removed link world
Joints:
- removed joint world_fixed

Commit message: change source

File: urdf/TFtest.urdf (robot description, URDF)
Before this commit: robot box, 2 links, 1 joints
Joints:
- joint world_fixed: origin xyz=0 0 0 rpy=0 0 0 -> xyz=0 0 0.0 rpy=0 0 0

File: urdf/abc.urdf (robot description, URDF)
Before this commit: robot box, 2 links, 1 joints
Links:
- removed link world
- link arrow: mass 100 -> 0.001; geometry collision mesh filename=meshes/abc.stl scale=0.01 0.01 0.01; visual mesh filename=meshes/abc.stl scale=0.01 0.01 0.01
Joints:
- removed joint world_fixed

File: urdf/box2.urdf (robot description, URDF)
Before this commit: robot box, 1 links, 0 joints
Links:
- added link ft_sensor, mass 10; collision box size=0.5 0.5 0.5; visual box size=0.5 0.5 0.5
- added link world
Joints:
- added joint FT_joint: type floating, parent ft_sensor, child box, origin xyz=0 0 0.75 rpy=0 0 0
- added joint world_fixed: type fixed, parent world, child ft_sensor, origin xyz=0 0 0.25 rpy=0 0 0
