Commit message: change source

File: urdf/box.urdf (robot description, URDF)
Before this commit: robot box, 2 links, 1 joints
Links:
- link box: geometry collision box size=1 3 3; visual box size=1 3 3

File: urdf/kr210l150_link.urdf (robot description, URDF)
Before this commit: robot kuka_kr210, 10 links, 9 joints
Links:
- removed link rail_link
Joints:
- removed joint rail_joint
- joint world_fixed: child rail_link -> base_link

Commit message: change source

File: urdf/box.urdf (robot description, URDF)
Before this commit: robot box, 1 links, 0 joints
Links:
- removed link box
- added link end
- added link ft_sensor, mass 100; collision box size=1 1 1; visual box size=1 1 1
Joints:
- added joint joint: type floating, parent ft_sensor, child end, origin xyz=0 0 1 rpy=0 0 0

File: urdf/box2.urdf (robot description, URDF)
Before this commit: robot box, 3 links, 2 joints
Links:
- added link end
Joints:
- added joint joint: type floating, parent ft_sensor, child end, origin xyz=0 0 0.25 rpy=0 0 0
- joint FT_joint: origin xyz=0 0 0.75 rpy=0 0 0 -> xyz=0 0 0.5 rpy=0 0 0; parent ft_sensor -> end

File: urdf/kr210l150.urdf (robot description, URDF)
Before this commit: robot kuka_kr210, 9 links, 8 joints
Links:
- removed link eef
- added link box, mass 100; collision box size=1 1 1; visual box size=1 1 1
Joints:
- joint r_fixed_eef: axis 0 0 1 -> 0 0 0; child eef -> box; origin xyz=0 0 0 rpy=0 0 0 -> xyz=0.5 0.0 0.0 rpy=0 0 0
