Commit message: change source

File: urdf/sphere.urdf (robot description, URDF)
Before this commit: robot box, 2 links, 1 joints
Links:
- added link box, mass 100; collision mesh filename=meshes/sphere.stl scale=1 1 1; visual mesh filename=meshes/sphere.stl scale=1 1 1
- added link world
- link ft_sensor: mass 100 -> 10; geometry collision box size=0.5 0.5 0.5; visual box size=0.5 0.5 0.5
Joints:
- added joint FT_joint: type floating, parent end, child box, origin xyz=0 0 1 rpy=0 0 0
- added joint world_fixed: type fixed, parent world, child ft_sensor, origin xyz=0 0 0.25 rpy=0 0 0
- joint joint: origin xyz=0 0 1 rpy=0 0 0 -> xyz=0 0 0.25 rpy=0 0 0
