Commit message: change source

File: urdf/abc.urdf (robot description, URDF)
Before this commit: robot box, 1 links, 0 joints
Links:
- link arrow: mass 0.001 -> 1; geometry collision mesh filename=meshes/abc.stl scale=0.02 0.02 0.01; visual mesh filename=meshes/abc.stl scale=0.02 0.02 0.01

File: urdf/box.urdf (robot description, URDF)
Before this commit: robot box, 2 links, 1 joints
Links:
- removed link ft_sensor
- added link box, mass 100; collision box size=1.5 1.5 0.5; visual box size=1.5 1.5 0.5
Joints:
- joint joint: parent ft_sensor -> box

File: urdf/box2.urdf (robot description, URDF)
Before this commit: robot box, 4 links, 3 joints
Links:
- removed link end
- added link link1
- link box: geometry collision box size=1.5 1.5 0.5; visual box size=1.5 1.5 0.5
Joints:
- removed joint FT_joint
- removed joint joint
- added joint joint1: type floating, parent link1, child ft_sensor, origin xyz=0 0 0.25 rpy=0 0 0
- added joint joint2: type floating, parent ft_sensor, child box, origin xyz=0 0 0.5 rpy=0 0 0
- joint world_fixed: child ft_sensor -> link1; origin xyz=0 0 0.25 rpy=0 0 0 -> xyz=0 0 0.0 rpy=0 0 0

File: urdf/kr210l150.urdf (robot description, URDF)
Before this commit: robot kuka_kr210, 9 links, 8 joints
Links:
- link box: geometry collision box size=1.5 1.5 0.5; visual box size=1.5 1.5 0.5
- link link_2: geometry collision mesh filename=C:/Users/whj03/Desktop/admittance/urdf/meshes/kr210l150/col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; visual mesh filename=C:/Users/whj03/Desktop/admittance/urdf/meshes/kr210l150/col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
Joints:
- joint r_fixed_eef: origin xyz=0.5 0.0 0.0 rpy=0 0 0 -> xyz=0.25 0.0 0.0 rpy=0 0 0

File: urdf/sphere.urdf (robot description, URDF)
Before this commit: robot box, 4 links, 3 joints
Links:
- removed link box
- removed link world
- link ft_sensor: mass 10 -> 100; geometry collision box size=1 1 1; visual box size=1 1 1
Joints:
- removed joint FT_joint
- removed joint world_fixed
- joint joint: origin xyz=0 0 0.25 rpy=0 0 0 -> xyz=0 0 1 rpy=0 0 0
